File: V2/ElectronPhotonTestHarness.brd (EAGLE design)
At the start: 100 x 133 mm, 43 parts, among them IC1 7805TV, Q1 200mA/50V, Q2 200mA/50V, U1 ELECTRONDUALNAMED, U2 UnderTest

Commit message: Tidy up for main test harness board.
Made test top (well middle) board for Pogo pins to rest in.
Parts:
- removed U$4: RELAYSONGLE, Particle:SRD-5VDC-SL-C
- JP4: value (none) -> FTDI Serial Output
- JP5: value (none) -> TestConnector
Routing:
- net VIN_TEST: track 176.4 -> 177.6 mm
Changed lines of the file:
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@@
 <setting verticaltext="up"/>
 </settings>
-<grid distance="0.25" unitdist="mm" unit="mm" style="lines" multiple="1" display="yes" altdistance="0.0125" altunitdist="inch" altunit="inch"/>
+<grid distance="0.025" unitdist="inch" unit="inch" style="lines" multiple="1" display="yes" altdistance="0.0125" altunitdist="inch" altunit="inch"/>
 <layers>
 <layer number="1" name="Top" color="4" fill="1" visible="yes" active="yes"/>
@@
 <text x="87.3125" y="68.2625" size="1.778" layer="25">B1</text>
 <text x="87.3125" y="71.4375" size="1.778" layer="25">PASS</text>
-<text x="64.77" y="102.235" size="1.016" layer="25" font="vector">3v3 FTDI</text>
-<text x="57.15" y="65.405" size="1.27" layer="25" font="vector">EXT Test Input</text>
+<text x="71.73" y="105.015" size="1.016" layer="25" font="vector" rot="R180">3v3 FTDI</text>
+<text x="56.9" y="63.905" size="1.27" layer="25" font="vector">EXT Test Input</text>
 <text x="34.925" y="116.84" size="1.016" layer="25" font="vector">+5V</text>
 <text x="40.005" y="116.84" size="1.016" layer="25" font="vector">GND</text>
@@
 <element name="H3" library="holes" package="3,2" value="MOUNT-HOLE3.2" x="4" y="96" locked="yes"/>
 <element name="H4" library="holes" package="3,2" value="MOUNT-HOLE3.2" x="96" y="96" locked="yes"/>
-<element name="JP1" library="SparkFun-Connectors" package="2X6" value="2X6 FEMALE" x="66.675" y="24.765" rot="R270">
+<element name="JP1" library="SparkFun-Connectors" package="2X6" value="2X6 FEMALE" x="66.675" y="24.765" smashed="yes" rot="R270">
 <attribute name="PROD_ID" value="CONN-12423" x="66.675" y="24.765" size="1.778" layer="27" rot="R270" display="off"/>
-</element>
-<element name="JP2" library="SparkFun-Connectors" package="2X6" value="2X6 FEMALE" x="31.115" y="24.765" rot="R270">
+<attribute name="NAME" x="65.715" y="8.87" size="1.27" layer="25" ratio="10"/>
+</element>
+<element name="JP2" library="SparkFun-Connectors" package="2X6" value="2X6 FEMALE" x="31.115" y="24.765" smashed="yes" rot="R270">
 <attribute name="PROD_ID" value="CONN-12423" x="31.115" y="24.765" size="1.778" layer="27" rot="R270" display="off"/>
+<attribute name="NAME" x="30.215" y="8.81" size="1.27" layer="25" ratio="10"/>
 </element>
 <element name="R1" library="SparkFun-Resistors" package="1206" value="" x="78.105" y="66.04" smashed="yes" rot="R180">
@@
 </element>
 <element name="U$2" library="Particle" package="SRD-5VDC-SL-C" value="RELAYSONGLE" x="83.185" y="114.3" rot="R90"/>
-<element name="H5" library="holes" package="3,2" value="MOUNT-HOLE3.2" x="73.5" y="50"/>
-<element name="H6" library="holes" package="3,2" value="MOUNT-HOLE3.2" x="26.5" y="50"/>
+<element name="H5" library="holes" package="3,2" value="MOUNT-HOLE3.2" x="73.5" y="50" locked="yes"/>
+<element name="H6" library="holes" package="3,2" value="MOUNT-HOLE3.2" x="26.5" y="50" locked="yes"/>
 <element name="D8" library="SparkFun-DiscreteSemi" package="SMA-DIODE" value="MBRA140" x="17.145" y="130.175" smashed="yes">
 <attribute name="PROD_ID" value="DIO-08053" x="17.145" y="130.175" size="2.54" layer="27" display="off"/>
@@
 <element name="Q2" library="SparkFun-DiscreteSemi" package="SOT23-3" value="200mA/50V" x="71.755" y="108.585" smashed="yes">
 <attribute name="PROD_ID" value="TRANS-00830" x="71.755" y="108.585" size="2.54" layer="27" display="off"/>
-<attribute name="NAME" x="72.5805" y="106.172" size="1.016" layer="25" rot="R180"/>
+<attribute name="NAME" x="69.5805" y="108.922" size="1.016" layer="25" rot="R180"/>
 </element>
 <element name="JP3" library="SparkFun-Connectors" package="SCREWTERMINAL-5MM-2" value="" x="4.445" y="125.095" smashed="yes" rot="R90">
@@
 <attribute name="VALUE" x="3.175" y="123.825" size="0.4064" layer="27" rot="R90"/>
 </element>
-<element name="H7" library="holes" package="3,2" value="MOUNT-HOLE3.2" x="26.5" y="4"/>
-<element name="H8" library="holes" package="3,2" value="MOUNT-HOLE3.2" x="73.5" y="4"/>
+<element name="H7" library="holes" package="3,2" value="MOUNT-HOLE3.2" x="26.5" y="4" locked="yes"/>
+<element name="H8" library="holes" package="3,2" value="MOUNT-HOLE3.2" x="73.5" y="4" locked="yes"/>
 <element name="U3" library="SparkFun-PowerIC" package="SOT223" value="" x="53.34" y="127.635" smashed="yes" rot="R270">
 <attribute name="PROD_ID" value="VREG-08170" x="53.34" y="127.635" size="2.54" layer="27" rot="R270" display="off"/>
@@
 <attribute name="VALUE" x="53.1495" y="128.7145" size="0.4064" layer="27" rot="R270"/>
 </element>
-<element name="JP4" library="SparkFun-Connectors" package="1X06" value="" x="75.565" y="99.06" smashed="yes" rot="R180">
+<element name="JP4" library="SparkFun-Connectors" package="1X06" value="FTDI Serial Output" x="75.565" y="99.06" smashed="yes" rot="R180">
 <attribute name="PROD_ID" value="CONN-08437" x="75.565" y="99.06" size="2.54" layer="27" rot="R180" display="off"/>
-<attribute name="VALUE" x="76.835" y="102.235" size="1.27" layer="27" rot="R180"/>
-</element>
-<element name="JP5" library="SparkFun-Connectors" package="1X06" value="" x="57.785" y="68.58" smashed="yes">
+<attribute name="VALUE" x="79.085" y="103.735" size="1.27" layer="27" rot="R180"/>
+</element>
+<element name="JP5" library="SparkFun-Connectors" package="1X06" value="TestConnector" x="57.785" y="68.58" smashed="yes">
 <attribute name="PROD_ID" value="CONN-08437" x="57.785" y="68.58" size="1.016" layer="27" font="vector" display="off"/>
 <attribute name="VALUE" x="56.515" y="65.405" size="1.27" layer="27"/>
@@
 </element>
 <element name="U$3" library="Particle" package="SRD-5VDC-SL-C" value="RELAYSONGLE" x="17.78" y="113.665" rot="R90"/>
-<element name="U$4" library="Particle" package="SRD-5VDC-SL-C" value="RELAYSONGLE" x="-15.875" y="-39.37"/>
 </elements>
 <signals>
@@
 <wire x1="45.085" y1="91.44" x2="45.085" y2="88.9" width="0.4064" layer="1"/>
 <wire x1="45.085" y1="88.9" x2="50.8" y2="83.185" width="0.4064" layer="1"/>
-<wire x1="50.8" y1="83.185" x2="90.805" y2="83.185" width="0.4064" layer="1"/>
-<wire x1="90.805" y1="83.185" x2="90.805" y2="41.91" width="0.4064" layer="1"/>
+<wire x1="50.8" y1="83.185" x2="90.17" y2="83.185" width="0.4064" layer="1"/>
+<wire x1="90.17" y1="83.185" x2="90.805" y2="82.55" width="0.4064" layer="1"/>
+<wire x1="90.805" y1="82.55" x2="90.805" y2="41.91" width="0.4064" layer="1"/>
 <wire x1="90.805" y1="41.91" x2="88.9" y2="40.005" width="0.4064" layer="1"/>
 <wire x1="88.9" y1="40.005" x2="61.595" y2="40.005" width="0.4064" layer="1"/>
@@
 <wire x1="38.735" y1="55.245" x2="41.275" y2="55.245" width="0.4064" layer="1"/>
 <contactref element="R2" pad="2"/>
-<wire x1="41.275" y1="55.245" x2="16.51" y2="55.245" width="1.27" layer="16"/>
-<wire x1="16.51" y1="55.245" x2="13.97" y2="57.15" width="1.27" layer="16"/>
-<wire x1="13.97" y1="57.15" x2="13.97" y2="106.5784" width="1.27" layer="16"/>
+<wire x1="41.275" y1="55.245" x2="13.01" y2="55.245" width="1.27" layer="16"/>
+<wire x1="13.01" y1="55.245" x2="11.72" y2="57.4" width="1.27" layer="16"/>
+<wire x1="11.72" y1="57.4" x2="11.72" y2="106.8284" width="1.27" layer="16"/>
 <wire x1="76.705" y1="75.565" x2="73.53" y2="78.105" width="0.6096" layer="1"/>
-<wire x1="73.53" y1="78.105" x2="14.605" y2="78.105" width="0.6096" layer="1"/>
-<wire x1="14.605" y1="78.105" x2="11.43" y2="81.28" width="0.6096" layer="1"/>
-<wire x1="11.43" y1="81.28" x2="11.4681" y2="107.4644" width="0.6096" layer="1"/>
+<wire x1="73.53" y1="78.105" x2="14.26" y2="78.105" width="0.6096" layer="1"/>
 <contactref element="U$3" pad="OPEN"/>
 <wire x1="11.4681" y1="107.4644" x2="11.5425" y2="107.39" width="0.6096" layer="1"/>
 <wire x1="11.5425" y1="107.39" x2="11.905" y2="107.39" width="0.6096" layer="1"/>
-<wire x1="13.97" y1="106.5784" x2="13.1584" y2="107.39" width="1.27" layer="16"/>
-<wire x1="13.1584" y1="107.39" x2="11.905" y2="107.39" width="1.27" layer="16"/>
+<wire x1="11.72" y1="106.8284" x2="11.9084" y2="107.39" width="1.27" layer="16"/>
+<wire x1="11.9084" y1="107.39" x2="11.905" y2="107.39" width="1.27" layer="16"/>
+<wire x1="14.26" y1="78.105" x2="11.72" y2="80.645" width="0.6096" layer="1"/>
+<wire x1="11.72" y1="80.645" x2="11.72" y2="107.205" width="0.6096" layer="1"/>
+<wire x1="11.72" y1="107.205" x2="11.905" y2="107.39" width="0.6096" layer="1"/>
 </signal>
 <signal name="A0">
